File: modules/DrokPowerSupply/DrokPowerSupply.kicad_pcb (KiCad board)
At the start: 2 copper layers, 28.2 x 23 mm, 5 parts, among them J1 Input, J2 Drok PS, J3 Vout, J4 Gnd

Commit message: Tweaked
Parts:
- J3: value Vout -> +
- J4: value Gnd -> -
- moved REF** 1.20 mm to (134.0, 88.8)
- moved J2 1.20 mm to (127.7, 93.4)
Connections:
- REF** pad 1: (no net) -> /GND
Routing:
- net /GND: track 24.8 -> 0.00 mm
Changed lines of the file:
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@@
   (net 4 "/VOUT")
   (footprint "Connector_PinSocket_2.54mm:PinSocket_1x04_P2.54mm_Horizontal" (layer "F.Cu")
-    (at 127.65 94.6 90)
+    (at 127.65 93.4 90)
     (descr "Through hole angled socket strip, 1x04, 2.54mm pitch, 8.51mm socket length, single row (from Kicad 4.0.7), script generated")
     (tags "Through hole angled socket strip THT 1x04 2.54mm single row")
@@
       (effects (font (size 1 1) (thickness 0.15)))
     )
-    (fp_text user "DROK" (at -12.065 3.81 unlocked) (layer "F.SilkS")
-      (effects (font (size 1 1) (thickness 0.15)))
+    (fp_text user "Vout" (at -10.85 7.6 270 unlocked) (layer "F.SilkS")
+      (effects (font (size 1 1) (thickness 0.15)) (justify left))
+    )
+    (fp_text user "Gnd" (at -10.85 5.1 270 unlocked) (layer "F.SilkS")
+      (effects (font (size 1 1) (thickness 0.15)) (justify left))
+    )
+    (fp_text user "Vin" (at -10.85 2.6 270 unlocked) (layer "F.SilkS")
+      (effects (font (size 1 1) (thickness 0.15)) (justify left))
+    )
+    (fp_text user "En" (at -10.85 0.1 270 unlocked) (layer "F.SilkS")
+      (effects (font (size 1 1) (thickness 0.15)) (justify left))
     )
     (fp_text user "${REFERENCE}" (at -5.775 3.81) (layer "F.Fab") hide
@@
   )
   (footprint "Connector_PinHeader_2.54mm:PinHeader_1x08_P2.54mm_Vertical" (layer "F.Cu")
-    (at 140 88)
+    (at 139.96 88)
     (descr "Through hole straight pin header, 1x08, 2.54mm pitch, single row")
     (tags "Through hole pin header THT 1x08 2.54mm single row")
@@
       (effects (font (size 1 1) (thickness 0.15)))
     )
-    (fp_text value "Vout" (at -1 20) (layer "F.SilkS")
+    (fp_text value "+" (at 0 20) (layer "F.SilkS")
       (effects (font (size 1 1) (thickness 0.15)))
     )
@@
   )
   (footprint "Connector_PinHeader_2.54mm:PinHeader_1x08_P2.54mm_Vertical" (layer "F.Cu")
-    (at 142.54 88)
+    (at 142.5 88)
     (descr "Through hole straight pin header, 1x08, 2.54mm pitch, single row")
     (tags "Through hole pin header THT 1x08 2.54mm single row")
@@
       (effects (font (size 1 1) (thickness 0.15)))
     )
-    (fp_text value "Gnd" (at -0.04 20) (layer "F.SilkS")
+    (fp_text value "-" (at -0.04 20) (layer "F.SilkS")
       (effects (font (size 1 1) (thickness 0.15)))
     )
@@
   )
   (footprint "MountingHole:MountingHole_2.5mm_Pad" locked (layer "F.Cu")
-    (at 134 90)
+    (at 134 88.8)
     (descr "Mounting Hole 2.5mm")
     (tags "mounting hole 2.5mm")
@@
     (fp_circle (center 0 0) (end 2.5 0) (layer "Cmts.User") (width 0.15) (fill none))
     (fp_circle (center 0 0) (end 2.75 0) (layer "F.CrtYd") (width 0.05) (fill none))
-    (pad "1" thru_hole circle locked (at 0 0) (size 5 5) (drill 2.5) (layers *.Cu *.Mask))
-  )
+    (pad "1" thru_hole circle locked (at 0 0) (size 5 5) (drill 2.5) (layers *.Cu *.Mask)
+      (net 2 "/GND"))
+  )
+  (gr_line (start 124 108.25) (end 125 108.25) (layer "F.SilkS") (width 0.15))
+  (gr_line (start 124 97.75) (end 125 97.75) (layer "F.SilkS") (width 0.15))
+  (gr_line (start 125 97.25) (end 125 93.5) (layer "F.SilkS") (width 0.15))
+  (gr_line (start 124 86.75) (end 125 86.75) (layer "F.SilkS") (width 0.15))
+  (gr_line (start 125 86.75) (end 125 90.75) (layer "F.SilkS") (width 0.15))
+  (gr_line (start 125 97.75) (end 125 101.25) (layer "F.SilkS") (width 0.15))
+  (gr_line (start 124 97.25) (end 125 97.25) (layer "F.SilkS") (width 0.15))
+  (gr_line (start 125 108.25) (end 125 104.25) (layer "F.SilkS") (width 0.15))
   (gr_rect (start 107.23 110.96) (end 109.77 113.5) (layer "Dwgs.User") (width 0.2) (fill none))
+  (gr_line (start 137.6 93.4) (end 125.6 93.4) (layer "Dwgs.User") (width 0.15))
   (gr_rect (start 116.25 86) (end 144.5 109) (layer "Edge.Cuts") (width 0.1) (fill none))
-  (gr_text "DrokPowerSupply v1" (at 130.5 106.5) (layer "B.SilkS")
+  (gr_text "DrokPowerSupply\nv1" (at 131.5 97.75) (layer "B.SilkS")
     (effects (font (size 1 1) (thickness 0.15)) (justify mirror))
   )
@@
     (style (thickness 0.1) (arrow_length 1.27) (text_position_mode 0) (extension_height 0.58642) (extension_offset 0.5) keep_text_aligned)
   )
-  (segment (start 130.19 93.1032) (end 125.8368 88.75) (width 2.032) (layer "F.Cu") (net 1))
+  (segment (start 130.2 93.39) (end 130.2 90.9) (width 2.032) (layer "F.Cu") (net 1))
   (segment (start 120.5 92.25) (end 120.5 95.75) (width 2.032) (layer "F.Cu") (net 1))
-  (segment (start 130.19 94.6) (end 130.19 93.1032) (width 2.032) (layer "F.Cu") (net 1))
   (segment (start 120.5 88.75) (end 120.5 92.25) (width 2.032) (layer "F.Cu") (net 1))
-  (segment (start 125.8368 88.75) (end 120.5 88.75) (width 2.032) (layer "F.Cu") (net 1))
-  (segment (start 120.5 102.75) (end 120.5 106.25) (width 2.032) (layer "F.Cu") (net 2))
-  (segment (start 142.54 90.54) (end 142.54 93.08) (width 2.032) (layer "F.Cu") (net 2))
-  (segment (start 142.54 98.16) (end 142.54 100.7) (width 2.032) (layer "F.Cu") (net 2))
-  (segment (start 142.54 100.7) (end 142.54 103.24) (width 2.032) (layer "F.Cu") (net 2))
-  (segment (start 142.54 88) (end 142.54 90.54) (width 2.032) (layer "F.Cu") (net 2))
-  (segment (start 120.5 99.25) (end 120.5 102.75) (width 2.032) (layer "F.Cu") (net 2))
-  (segment (start 142.54 95.62) (end 142.54 98.16) (width 2.032) (layer "F.Cu") (net 2))
-  (segment (start 142.54 103.24) (end 142.54 105.78) (width 2.032) (layer "F.Cu") (net 2))
-  (segment (start 142.54 93.08) (end 142.54 95.62) (width 2.032) (layer "F.Cu") (net 2))
-  (segment (start 140 103.24) (end 140 105.78) (width 2.032) (layer "F.Cu") (net 4))
-  (segment (start 140 88) (end 140 90.54) (width 2.032) (layer "F.Cu") (net 4))
-  (segment (start 138.98 94.6) (end 140 95.62) (width 2.032) (layer "F.Cu") (net 4))
-  (segment (start 140 90.54) (end 140 93.08) (width 2.032) (layer "F.Cu") (net 4))
-  (segment (start 135.27 94.6) (end 138.98 94.6) (width 2.032) (layer "F.Cu") (net 4))
-  (segment (start 140 100.7) (end 140 103.24) (width 2.032) (layer "F.Cu") (net 4))
-  (segment (start 140 93.08) (end 140 95.62) (width 2.032) (layer "F.Cu") (net 4))
-  (segment (start 140 95.62) (end 140 98.16) (width 2.032) (layer "F.Cu") (net 4))
-  (segment (start 140 98.16) (end 140 100.7) (width 2.032) (layer "F.Cu") (net 4))
+  (segment (start 130.19 93.4) (end 130.2 93.39) (width 2.032) (layer "F.Cu") (net 1))
+  (segment (start 128.05 88.75) (end 120.5 88.75) (width 2.032) (layer "F.Cu") (net 1))
+  (segment (start 130.2 90.9) (end 128.05 88.75) (width 2.032) (layer "F.Cu") (net 1))
+  (segment (start 139.96 100.7) (end 139.96 103.24) (width 2.032) (layer "F.Cu") (net 4))
+  (segment (start 135.27 93.4) (end 139.64 93.4) (width 2.032) (layer "F.Cu") (net 4))
+  (segment (start 139.96 95.62) (end 139.96 98.16) (width 2.032) (layer "F.Cu") (net 4))
+  (segment (start 139.64 93.4) (end 139.96 93.08) (width 2.032) (layer "F.Cu") (net 4))
+  (segment (start 139.96 88) (end 139.96 90.54) (width 2.032) (layer "F.Cu") (net 4))
+  (segment (start 139.96 98.16) (end 139.96 100.7) (width 2.032) (layer "F.Cu") (net 4))
+  (segment (start 139.96 103.24) (end 139.96 105.78) (width 2.032) (layer "F.Cu") (net 4))
+  (segment (start 139.96 93.08) (end 139.96 95.62) (width 2.032) (layer "F.Cu") (net 4))
+  (segment (start 139.96 90.54) (end 139.96 93.08) (width 2.032) (layer "F.Cu") (net 4))
   (zone (net 2) (net_name "/GND") (layers F&B.Cu) (hatch edge 0.508)
-    (connect_pads (clearance 0.508))
+    (connect_pads (clearance 0.381))
     (min_thickness 0.254) (filled_areas_thickness no)
     (fill yes (thermal_gap 0.508) (thermal_bridge_width 0.508))
