File: modules/19PinHeader/19PinHeader.kicad_pcb (KiCad board)
At the start: 2 copper layers, 8.9 x 64.8 mm, 4 parts, among them J1 Conn_01x19, J2 Conn_01x19

Commit message: Changed REF names
Parts:
- J1: value Conn_01x19 -> Socket
- J2: value Conn_01x19 -> Header
Changed lines of the file:
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@@
       (effects (font (size 1 1) (thickness 0.15)))
     )
-    (fp_text value "Conn_01x19" (at 0 48.05) (layer "F.Fab") hide
+    (fp_text value "Header" (at 0 48.05) (layer "F.Fab") hide
       (effects (font (size 1 1) (thickness 0.15)))
     )
@@
       (effects (font (size 1 1) (thickness 0.15)))
     )
-    (fp_text value "Conn_01x19" (at 0 48.49) (layer "F.Fab") hide
+    (fp_text value "Socket" (at 0 48.49) (layer "F.Fab") hide
       (effects (font (size 1 1) (thickness 0.15)))
     )
